File: _saved_bed_sensor.sch (KiCad schematic (older format))
At the start: 15 parts

Commit message: updated schematic
Parts:
- removed J?: Conn_01x02, symbol Connector:Conn_01x02
- removed RV?: POT, symbol device:POT
- removed SW?: SW_DPST_x2, symbol foot_sensor-rescue:SW_DPST_x2
- removed U?: CFAH0802D-YYH-JP, symbol Crystalfontz:CFAH0802D-YYH-JP
- removed U?: SPX3819M5-L-3-3, TO_SOT_Packages_SMD:SOT-23-5, symbol foot_sensor-rescue:SPX3819M5-L-3-3
- added C2: 10nF, Capacitor_SMD:C_0603_1608Metric, symbol Device:C
- added C5: .1uF, Capacitor_SMD:C_0603_1608Metric, symbol Device:C
- added C6: 1uF, Capacitor_SMD:C_0603_1608Metric, symbol Device:C
- added C7: 10uF, Capacitor_SMD:C_0603_1608Metric, symbol Device:C
- added J1: Conn_01x02, Connector_PinHeader_2.54mm:PinHeader_1x02_P2.54mm_Vertical, symbol Connector_Generic:Conn_01x02
- added J4: Conn_01x02, components:JSTPH2, symbol Connector_Generic:Conn_01x02
- added L1: 10uH, Inductors_SMD:L_Taiyo-Yuden_NR-40xx, symbol Device:L_Core_Ferrite_Small
- added Q2, Q3: BSS138, Package_TO_SOT_SMD:SOT-23, symbol Transistor_FET:BSS138
- added R1, R2, R6, R7: 10k, Resistor_SMD:R_0805_2012Metric, symbol Device:R
- added RV1: 10K, Potentiometers:Potentiometer_Trimmer_ACP_CA9h2.5_Vertical_Px2.5mm_Py5.0mm, symbol Device:R_POT
- added SW1: SW_SPST, components:SW_CuK_OS102011MA1QN1_SPDT_Angled, symbol Switch:SW_SPST
- added U1: MIC5205-3.3, Package_TO_SOT_SMD:SOT-23-5, symbol Regulator_Linear:MIC5205-3.3
- added U2: MPU-9250, Package_DFN_QFN:QFN-24-1EP_3x3mm_P0.4mm_EP1.75x1.6mm, symbol Sensor_Motion:MPU-9250
- added U3: TXB0104D, Package_SO:SOIC-14_3.9x8.7mm_P1.27mm, symbol Logic_LevelTranslator:TXB0104D
- added U4: LTC3525-5, Package_TO_SOT_SMD:SOT-363_SC-70-6, symbol Regulator_Switching:LTC3525-5
- added U5: CFAH0802D-YYH-JP, components:CFAH0802D-YYH-JP, symbol Crystalfontz:CFAH0802D-YYH-JP
- BZ1: renamed from BZ?; footprint (none) -> components:PS1240P02BT
- C1: renamed from C?; value CP1 -> 10uF; footprint (none) -> Capacitors_Tantalum_SMD:CP_Tantalum_Case-T_EIA-3528-12_Reflow
- C3: renamed from C?; value CP1 -> 10uF; footprint (none) -> Capacitors_Tantalum_SMD:CP_Tantalum_Case-B_EIA-3528-21_Reflow
- C4: renamed from C?; value C -> .1uF; footprint (none) -> Capacitor_SMD:C_0603_1608Metric
- D1: renamed from D?; footprint (none) -> LED_SMD:LED_0603_1608Metric
- D2: renamed from D?; footprint (none) -> Diode_SMD:D_0603_1608Metric
- Q1: renamed from Q?; footprint Package_TO_SOT_THT:TO-39-3 -> Package_TO_SOT_SMD:SOT-723
- R3: renamed from R?; value R -> 10k; footprint (none) -> Resistor_SMD:R_0805_2012Metric
- R4: renamed from R?; value R -> 1K; footprint (none) -> Resistor_SMD:R_0805_2012Metric
- R5: renamed from R?; footprint (none) -> Resistor_SMD:R_0805_2012Metric
Connections:
- net labels added: +5V, SCL_MPU, SDA_MPU
- wire segments 20 -> 53
- no-connect marks 0 -> 2
Other:
- moved on the sheet: BZ1, C1, C3, C4, D1, D2, Q1, R3, R4, R5
