File: Ardunio.sch (KiCad schematic (older format))
At the start: 11 parts, among them J2 Conn_01x06, J3 ISP, U6 ATMEGA328-AU, Y1 Crystal_GND2

Commit message: updated design
Parts:
- removed U6: ATMEGA328-AU, Package_QFP:TQFP-32_7x7mm_P0.8mm, symbol MCU_Atmel_ATMEGA:ATMEGA328-AU
- added U6: ATMEGA328-AU, Housings_QFP:TQFP-32_7x7mm_Pitch0.8mm, symbol atmel:ATMEGA328-AU
Connections:
- net +3V3: now also U6.18 (AVCC), U6.4 (VCC), U6.6 (VCC)
- net A0: now also U6.23 ((PCINT8/ADC0)PC0)
- net A1: now also U6.24 ((PCINT9/ADC1)PC1)
- net A2: now also U6.25 ((PCINT10/ADC2)PC2)
- net A3: now also U6.26 ((PCINT11/ADC3)PC3)
- net A6: now also U6.19 (ADC6)
- net A7: now also U6.22 (ADC7)
- net D10: now also U6.14 ((PCINT2/OC1B/~SS~)PB2)
- net D2: now also U6.32 ((PCINT18/INT0)PD2)
- net D3: now also U6.1 ((PCINT19/OC2B/INT1)PD3)
- net D4: now also U6.2 ((PCINT20/XCK/T0)PD4)
- net D5: now also U6.9 ((PCINT21/OC0B/T1)PD5)
- net D6: now also U6.10 ((PCINT22/OC0A/AIN0)PD6)
- net D7: now also U6.11 ((PCINT23/AIN1)PD7)
- net D8: now also U6.12 ((PCINT0/CLKO/ICP1)PB0)
- net D9: now also U6.13 ((PCINT1/OC1A)PB1)
- net GND: now also U6.21 (GND), U6.3 (GND), U6.5 (GND)
- net MISO: now also U6.16 ((PCINT4/MISO)PB4)
- net MOSI: now also U6.15 ((PCINT3/OC2A/MOSI)PB3)
- net RESET: now also U6.29 ((PCINT14/~RESET~)PC6)
- net RX1: now also U6.30 ((PCINT16/RXD)PD0)
- net SCK: now also U6.17 ((PCINT5/SCK)PB5)
- net SCL: now also U6.28 ((PCINT13/SCL/ADC5)PC5)
- net SDA: now also U6.27 ((PCINT12/SDA/ADC4)PC4)
- net TX0: now also U6.31 ((PCINT17/TXD)PD1)
- net at C9.1: now also U6.20 (AREF)
- net at Y1.3: now also U6.7 ((PCINT6/XTAL1/TOSC1)PB6)
- net at Y1.1: now also U6.8 ((PCINT7/XTAL2/TOSC2)PB7)
Changed lines of the file:
@@
 	5800 3500 6650 3500
-$Comp
-L MCU_Atmel_ATMEGA:ATMEGA328-AU U6
-U 1 1 5B120A6F
-P 4750 3150
-F 0 "U6" H 4800 4517 50  0000 C CNN
-F 1 "ATMEGA328-AU" H 4800 4426 50  0000 C CNN
-F 2 "Package_QFP:TQFP-32_7x7mm_P0.8mm" H 4750 3150 50  0001 C CIN
-F 3 "http://ww1.microchip.com/downloads/en/DeviceDoc/atmel-8271-8-bit-avr-microcontroller-atmega48a-48pa-88a-88pa-168a-168pa-328-328p_datasheet.pdf" H 4750 3150 50  0001 C CNN
-	1    4750 3150
-	1    0    0    -1
-$EndComp
 $Comp
 L Device:C C9
@@
 	-1   0    0    1
 $EndComp
+$Comp
+L atmel:ATMEGA328-AU U6
+U 1 1 5B11F80F
+P 4750 3150
+F 0 "U6" H 4800 4517 50  0000 C CNN
+F 1 "ATMEGA328-AU" H 4800 4426 50  0000 C CNN
+F 2 "Housings_QFP:TQFP-32_7x7mm_Pitch0.8mm" H 4750 3150 50  0001 C CIN
+F 3 "http://www.atmel.com/images/atmel-8271-8-bit-avr-microcontroller-atmega48a-48pa-88a-88pa-168a-168pa-328-328p_datasheet.pdf" H 4750 3150 50  0001 C CNN
+	1    4750 3150
+	1    0    0    -1
+$EndComp
 $EndSCHEMATC

Commit message: working out missing sd card`
Parts:
- J3: symbol Connector_Generic:Conn_02x03_Top_Bottom -> Connector_Generic:Conn_02x03_Odd_Even
- U6: symbol atmel:ATMEGA328-AU -> MCU_Atmel_ATMEGA:ATMEGA328-AU
Connections:
- net MOSI: now also J3.4 (Pin_4); no longer J3.5 (Pin_5)
- net RESET: now also J3.5 (Pin_5); no longer J3.3 (Pin_3)
- net SCK: now also J3.3 (Pin_3); no longer J3.2 (Pin_2)
- net VCC: now also J3.2 (Pin_2); no longer J3.4 (Pin_4)
Changed lines of the file:
@@
-$EndComp
-$Comp
-L Connector_Generic:Conn_02x03_Top_Bottom J3
-U 1 1 5B121CDB
-P 8250 1900
-F 0 "J3" H 8300 2217 50  0000 C CNN
-F 1 "ISP" H 8300 2126 50  0000 C CNN
-F 2 "Connector_PinHeader_2.54mm:PinHeader_2x03_P2.54mm_Vertical" H 8250 1900 50  0001 C CNN
-F 3 "~" H 8250 1900 50  0001 C CNN
-	1    8250 1900
-	1    0    0    -1
 $EndComp
 $Comp
@@
 $EndComp
 $Comp
-L atmel:ATMEGA328-AU U6
+L MCU_Atmel_ATMEGA:ATMEGA328-AU U6
 U 1 1 5B11F80F
 P 4750 3150
@@
 	1    0    0    -1
 $EndComp
+$Comp
+L Connector_Generic:Conn_02x03_Odd_Even J3
+U 1 1 5B121CDB
+P 8250 1900
+F 0 "J3" H 8300 2217 50  0000 C CNN
+F 1 "ISP" H 8300 2126 50  0000 C CNN
+F 2 "Connector_PinHeader_2.54mm:PinHeader_2x03_P2.54mm_Vertical" H 8250 1900 50  0001 C CNN
+F 3 "~" H 8250 1900 50  0001 C CNN
+	1    8250 1900
+	1    0    0    -1
+$EndComp
