File: hardware/Ardunio.sch (KiCad schematic (older format))
At the start: 11 parts, among them J2 Conn_01x06, J3 ISP, U3 ATMEGA328-AU, Y1 Crystal_GND2

Commit message: modified design slightly and fixed problems with layout
Parts:
- J2: footprint Connector_PinHeader_2.54mm:PinHeader_1x06_P2.54mm_Vertical -> Connector_PinHeader_2.00mm:PinHeader_1x06_P2.00mm_Vertical
Changed lines of the file:
@@
 F 0 "J2" H 7920 2625 50  0000 C CNN
 F 1 "Conn_01x06" H 7920 2716 50  0000 C CNN
-F 2 "Connector_PinHeader_2.54mm:PinHeader_1x06_P2.54mm_Vertical" H 8000 3150 50  0001 C CNN
+F 2 "Connector_PinHeader_2.00mm:PinHeader_1x06_P2.00mm_Vertical" H 8000 3150 50  0001 C CNN
 F 3 "~" H 8000 3150 50  0001 C CNN
 	1    8000 3150

Commit message: tweaked firmware for angle
Parts:
- U3: symbol MCU_Atmel_ATMEGA:ATMEGA328-AU -> bed_sensor-rescue:ATMEGA328-AU-MCU_Atmel_ATMEGA
Changed lines of the file:
@@
 EESchema Schematic File Version 4
 LIBS:bed_sensor-cache
-EELAYER 26 0
+EELAYER 29 0
 EELAYER END
 $Descr A4 11693 8268
@@
 $EndComp
 $Comp
-L MCU_Atmel_ATMEGA:ATMEGA328-AU U3
+L bed_sensor-rescue:ATMEGA328-AU-MCU_Atmel_ATMEGA U3
 U 1 1 5B216C7D
 P 4750 3150
