File: hardware/bed_sensor.sch (KiCad schematic (older format))
At the start: 22 parts, among them J1 Conn_01x02, J4 Conn_01x02, J5 DM3AT-SF-PEJM5, Q1 2N2219, SW1 SW_SPST, U1 MIC5205-3.3, U2 MPU-9250, U5 CFAH0802D-YYH-JP

Commit message: updated schematic removed old kicad design
Other:
- note added: "Ardunio\n"
- note added: "Display\n"
- note added: "MPU 9250\n"
- note added: "Power\n"
- note added: "SD card\n"
- note added: "Stimuli\n"
- moved on the sheet: BZ1, C2, C5, C6, D2, J1, J4, J5, Q1, R1, R2, R4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

Commit message: tweaked firmware for angle
Parts:
- U1: symbol Regulator_Linear:MIC5205-3.3 -> bed_sensor-rescue:MIC5205-3.3-Regulator_Linear
Changed lines of the file:
@@
 EESchema Schematic File Version 4
 LIBS:bed_sensor-cache
-EELAYER 26 0
+EELAYER 29 0
 EELAYER END
 $Descr A4 11693 8268
@@
 	1800 3150 1800 3300
 $Comp
-L Regulator_Linear:MIC5205-3.3 U1
+L bed_sensor-rescue:MIC5205-3.3-Regulator_Linear U1
 U 1 1 5B11C18F
 P 2650 1250
