File: hardware/bed-sensor.kicad_pcb (KiCad board)
At the start: 2 copper layers, 40 parts, among them J1 USB_B_Mini, J2 Conn_ARM_JTAG_SWD_10, J3 DM3AT-SF-PEJM5, SW1 SW_Push, U1 MCP73831-2-OT, U2 TLV70218_SOT23-5, U3 AP2112K-3.3, U4 MDBT50Q-1M, U6 ICM-20948, U7 BMP280

Commit message: started building board
Parts:
- added BZ1: Buzzer, Buzzer_Beeper:Buzzer_Murata_PKMCS0909E4000-R1, B.Cu at (125.3, -31.9)
- added D2: LED, Capacitor_SMD:C_0603_1608Metric, F.Cu at (130.5, -9.32)
- added J4: Conn_01x02, Connector_PinHeader_2.54mm:PinHeader_1x02_P2.54mm_Vertical, F.Cu at (131.7, -15.4)
- added Q1: Q_PMOS_GSD, digikey-footprints:SOT-23-3, F.Cu at (127.9, -19.3)
- added U5: PCA9306, Package_SO:VSSOP-8_2.3x2mm_P0.5mm, F.Cu at (117.6, -31.3)
- added Y1: 32.768, OPL_Crystal_Oscillator:X2-SMD-3.2X1.5X0.55MM, F.Cu at (124.9, -32.5)
- R1, R10, R11, R12, R13, R2, R5, R6, R7, R8, R9: footprint Resistor_SMD:R_0805_2012Metric -> Fuse:Fuse_0603_1608Metric
- R3, R4: footprint Resistor_SMD:R_0603_1608Metric -> Fuse:Fuse_0603_1608Metric
- moved C10 40.9 mm to (115.8, -12.1)
- moved C16 37.6 mm to (115.4, -32.1), turned to 270 degrees
- moved R6 37.0 mm to (132.3, -9.30), turned to 90 degrees
- moved R8 35.2 mm to (120.9, -33.1)
- moved C12 34.2 mm to (120.1, -30.8), turned to 270 degrees
- moved R9 32.5 mm to (116.6, -36.2), turned to 90 degrees
- moved C6 31.2 mm to (123.4, -19.5), turned to 270 degrees
- moved C15 30.1 mm to (116.0, -22.9)
- moved C11 29.4 mm to (116.0, -21.3)
- moved C7 29.3 mm to (127.2, -30.2), turned to 180 degrees
- moved R2 28.0 mm to (116.8, -14.4), turned to 90 degrees
- moved C2 27.2 mm to (132.3, -31.9)
- moved C3 25.2 mm to (119.6, -22.7)
- moved C9 25.0 mm to (115.0, -14.5), turned to 270 degrees
- moved D1 23.5 mm to (131.6, -18.4)
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Connections:
- J1 pad 4: Net-(J1-Pad4) -> (no net)
- J2 pad 8: Net-(J2-Pad8) -> (no net)
- J3 pad 1: Net-(J3-Pad1) -> (no net)
- J3 pad 8: Net-(J3-Pad8) -> (no net)
- J3 pad SWA: Net-(J3-PadSWA) -> (no net)
- J3 pad SWB: Net-(J3-PadSWB) -> (no net)
- U2 pad 4: Net-(U2-Pad4) -> (no net)
- U3 pad 4: Net-(U3-Pad4) -> (no net)
- U4 pad 1: Net-(U4-Pad1) -> GND
- U4 pad 10: Net-(U4-Pad10) -> (no net)
- U4 pad 11: Net-(U4-Pad11) -> (no net)
- U4 pad 12: Net-(U4-Pad12) -> (no net)
- U4 pad 13: Net-(U4-Pad13) -> (no net)
- U4 pad 14: Net-(U4-Pad14) -> (no net)
- U4 pad 15: Net-(U4-Pad15) -> GND
- U4 pad 16: Net-(U4-Pad16) -> (no net)
- U4 pad 19: Net-(U4-Pad19) -> SCL_MPU
- U4 pad 20: Net-(U4-Pad20) -> (no net)
- U4 pad 21: Net-(U4-Pad21) -> SDA_MPU
- U4 pad 22: SCL_MPU -> (no net)
- U4 pad 23: Net-(U4-Pad23) -> (no net)
- U4 pad 24: SDA_MPU -> (no net)
- U4 pad 26: Net-(U4-Pad26) -> (no net)
- U4 pad 27: Net-(U4-Pad27) -> (no net)
- U4 pad 29: Net-(U4-Pad29) -> (no net)
- U4 pad 3: Net-(U4-Pad3) -> (no net)
- U4 pad 31: Net-(U4-Pad31) -> (no net)
- U4 pad 33: Net-(U4-Pad15) -> GND
- U4 pad 38: Net-(U4-Pad38) -> (no net)
- U4 pad 4: Net-(U4-Pad4) -> (no net)
- U4 pad 41: Net-(U4-Pad41) -> (no net)
- U4 pad 42: Net-(U4-Pad42) -> (no net)
- U4 pad 43: Net-(U4-Pad43) -> (no net)
- U4 pad 44: Net-(U4-Pad44) -> (no net)
- U4 pad 45: Net-(U4-Pad45) -> (no net)
- U4 pad 46: Net-(U4-Pad46) -> (no net)
- U4 pad 48: Net-(U4-Pad48) -> (no net)
- U4 pad 5: Net-(U4-Pad5) -> (no net)
- U4 pad 50: Net-(U4-Pad50) -> (no net)
- U4 pad 52: Net-(U4-Pad52) -> (no net)
- U4 pad 54: Net-(U4-Pad54) -> (no net)
- U4 pad 56: Net-(U4-Pad56) -> (no net)
- U4 pad 6: Net-(U4-Pad6) -> (no net)
- U4 pad 60: Net-(U4-Pad60) -> (no net)
- U4 pad 61: Net-(U4-Pad61) -> (no net)
- U4 pad 7: Net-(U4-Pad7) -> (no net)
- U4 pad 8: Net-(U4-Pad8) -> (no net)
- U4 pad 9: Net-(U4-Pad9) -> (no net)
- U6 pad 12: Net-(U6-Pad12) -> (no net)
- U6 pad 19: Net-(U6-Pad19) -> (no net)
- U6 pad 21: Net-(U6-Pad21) -> (no net)
- U6 pad 7: Net-(U6-Pad7) -> (no net)
Routing:
- net VBUS: track 0.00 -> 48.0 mm
- net +3V3: track 0.00 -> 46.5 mm
- net RESET: track 0.00 -> 32.5 mm, vias 0 -> 2
- net SWCLK: track 0.00 -> 23.2 mm, vias 0 -> 2
- net SD_CS: track 0.00 -> 22.0 mm, vias 0 -> 1
- net SWDIO: track 0.00 -> 20.8 mm, vias 0 -> 2
- net SD_MOSI: track 0.00 -> 18.9 mm, vias 0 -> 1
- net SD_MISO: track 0.00 -> 18.6 mm, vias 0 -> 1
- net SWO: track 0.00 -> 18.0 mm, vias 0 -> 2
- net +1V8: track 0.00 -> 15.3 mm
- net +BATT: track 0.00 -> 15.1 mm
- net SD_SCK: track 0.00 -> 14.8 mm, vias 0 -> 1
- net BMP_SDA: track 0.00 -> 11.9 mm, vias 0 -> 2
- net SDA_MPU: track 0.00 -> 11.5 mm
- net SCL_MPU: track 0.00 -> 8.53 mm
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- added copper zone on B.Cu, net GND
Other:
- board outline added: 21.2 x 42.8 mm
- net class Default: trace_width 0.25 -> 0.2

Commit message: updated schematic
Parts:
- moved R2 3.03 mm to (116.5, -17.4), turned to 180 degrees
- moved C2 2.95 mm to (132.8, -29.0)
- moved C15 2.79 mm to (118.8, -22.7), turned to 90 degrees
- moved C10 2.49 mm to (116.8, -14.4), turned to 270 degrees
- moved U2 2.06 mm to (116.0, -20.4)
- moved C1 1.98 mm to (131.8, -26.1)
- moved C11 1.95 mm to (116.1, -23.2)
- moved C3 1.11 mm to (120.7, -22.5), turned to 90 degrees
- moved R8 0.51 mm to (120.4, -33.1)
- moved R3 0.50 mm to (132.8, -33.1)
- moved R4 0.50 mm to (132.9, -34.7)
- moved C14 0.45 mm to (121.3, -30.8)
- moved C12 0.45 mm to (119.7, -30.8)
- moved R1 0.22 mm to (125.1, -19.5)
- moved C9 0.10 mm to (115.0, -14.4)
Connections:
- J1 pad 4: (no net) -> Net-(J1-Pad4)
- J2 pad 8: (no net) -> Net-(J2-Pad8)
- J3 pad 1: (no net) -> Net-(J3-Pad1)
- J3 pad 8: (no net) -> Net-(J3-Pad8)
- J3 pad SWA: (no net) -> Net-(J3-PadSWA)
- J3 pad SWB: (no net) -> Net-(J3-PadSWB)
- R12 pad 2: +1V8 -> +3V3
- R13 pad 2: +1V8 -> +3V3
- U2 pad 4: (no net) -> Net-(U2-Pad4)
- U3 pad 4: (no net) -> Net-(U3-Pad4)
- U4 pad 10: (no net) -> Net-(U4-Pad10)
- U4 pad 11: (no net) -> Net-(U4-Pad11)
- U4 pad 12: (no net) -> Net-(U4-Pad12)
- U4 pad 13: (no net) -> Net-(U4-Pad13)
- U4 pad 14: (no net) -> Net-(U4-Pad14)
- U4 pad 16: (no net) -> Net-(U4-Pad16)
- U4 pad 20: (no net) -> Net-(U4-Pad20)
- U4 pad 22: (no net) -> Net-(U4-Pad22)
- U4 pad 23: (no net) -> Net-(U4-Pad23)
- U4 pad 24: (no net) -> Net-(U4-Pad24)
- U4 pad 26: (no net) -> Net-(U4-Pad26)
- U4 pad 27: (no net) -> Net-(U4-Pad27)
- U4 pad 29: (no net) -> Net-(U4-Pad29)
- U4 pad 3: (no net) -> Net-(U4-Pad3)
- U4 pad 31: (no net) -> Net-(U4-Pad31)
- U4 pad 38: (no net) -> Net-(U4-Pad38)
- U4 pad 4: (no net) -> Net-(U4-Pad4)
- U4 pad 41: (no net) -> Net-(U4-Pad41)
- U4 pad 42: (no net) -> Net-(U4-Pad42)
- U4 pad 43: (no net) -> Net-(U4-Pad43)
- U4 pad 44: (no net) -> Net-(U4-Pad44)
- U4 pad 45: (no net) -> Net-(U4-Pad45)
- U4 pad 46: (no net) -> Net-(U4-Pad46)
- U4 pad 48: (no net) -> Net-(U4-Pad48)
- U4 pad 5: (no net) -> Net-(U4-Pad5)
- U4 pad 50: (no net) -> Net-(U4-Pad50)
- U4 pad 52: (no net) -> Net-(U4-Pad52)
- U4 pad 54: (no net) -> Net-(U4-Pad54)
- U4 pad 56: (no net) -> Net-(U4-Pad56)
- U4 pad 6: (no net) -> Net-(U4-Pad6)
- U4 pad 60: (no net) -> Net-(U4-Pad60)
- U4 pad 61: (no net) -> Net-(U4-Pad61)
- U4 pad 7: (no net) -> Net-(U4-Pad7)
- U4 pad 8: (no net) -> Net-(U4-Pad8)
- U4 pad 9: (no net) -> Net-(U4-Pad9)
- U6 pad 12: (no net) -> Net-(U6-Pad12)
- U6 pad 19: (no net) -> Net-(U6-Pad19)
- U6 pad 21: (no net) -> Net-(U6-Pad21)
- U6 pad 7: (no net) -> Net-(U6-Pad7)
Routing:
- net GND: track 0.00 -> 107.0 mm, vias 0 -> 23
- net +3V3: track 46.5 -> 83.0 mm, vias 0 -> 6
- net USB_D+: track 0.00 -> 25.2 mm, vias 0 -> 2
- net USB_D-: track 0.00 -> 23.2 mm, vias 0 -> 2
- net +1V8: track 15.3 -> 37.6 mm
- net Net-(R6-Pad1): track 0.00 -> 17.8 mm, vias 0 -> 2
- net Net-(C3-Pad1): track 4.43 -> 20.2 mm, vias 0 -> 1
- net BUZZER: track 0.24 -> 10.2 mm, vias 0 -> 1
- net Net-(R11-Pad1): track 0.00 -> 8.46 mm, vias 0 -> 2
- net Net-(R10-Pad1): track 0.00 -> 4.32 mm
- net Net-(R5-Pad1): track 0.00 -> 4.18 mm
- net VBUS: track 48.0 -> 50.5 mm
- net Net-(R2-Pad1): track 0.20 -> 2.45 mm
- net Net-(D2-Pad1): track 0.00 -> 1.76 mm
- net SWO: track 18.0 -> 16.5 mm
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Other:
- board size 21.2 x 42.8 mm -> 21.3 x 43.2 mm
- rule pad_to_mask_clearance: 0.051 -> 0.03

Commit message: moved pin
Parts:
- moved J4 0.72 mm to (132.3, -15.7)
- moved R12 0.14 mm to (132.9, -38.4)
- moved R13 0.08 mm to (132.9, -40.0)
Connections:
- U4 pad 56: Net-(U4-Pad56) -> SD_CS
- U4 pad 59: SD_CS -> Net-(U4-Pad59)
Routing:
- net SD_CS: track 21.8 -> 18.6 mm
- net VBUS: track 50.5 -> 51.9 mm
- net +BATT: track 15.2 -> 14.6 mm
