File: hardware/bed-sensor.sch (KiCad schematic (older format))
At the start: 23 parts, among them J1 USB_B_Mini, J2 Conn_ARM_JTAG_SWD_10, Q1 Q_PMOS_DGS, U1 AP2112K-3.3, U2 MDBT50Q-1M, Y1 32.768

Commit message: added symbolds and started to lay out board
Parts:
- removed C3: CP_Small, symbol Device:CP_Small
- removed C6: CP, symbol Device:CP
- removed J1: USB_B_Mini, symbol Connector:USB_B_Mini
- removed J2: Conn_ARM_JTAG_SWD_10, Connector_PinHeader_1.27mm:PinHeader_2x05_P1.27mm_Vertical_SMD, symbol Connector:Conn_ARM_JTAG_SWD_10
- removed U1: AP2112K-3.3, Package_TO_SOT_SMD:SOT-23-5, symbol Regulator_Linear:AP2112K-3.3
- removed U2: MDBT50Q-1M, symbol extra:MDBT50Q-1M
- added BZ1: Buzzer, symbol Device:Buzzer
- added C10, C11: 1uF, Capacitor_SMD:C_0603_1608Metric, symbol Device:C_Small
- added C12: 100PF, Capacitor_SMD:C_0603_1608Metric, symbol Device:C_Small
- added C13, C14, C15, C16, C9: .1uF, Capacitor_SMD:C_0603_1608Metric, symbol Device:C_Small
- added C3, C6: 10uF, Capacitor_SMD:C_0805_2012Metric, symbol Device:C
- added J1: USB_B_Mini, Connectors:USB_Mini-B, symbol Connector_Specialized:USB_B_Mini
- added J2: Conn_ARM_JTAG_SWD_10, Connector_PinHeader_1.27mm:PinHeader_2x05_P1.27mm_Vertical_SMD, symbol Connector_Specialized:Conn_ARM_JTAG_SWD_10
- added J3: DM3AT-SF-PEJM5, extra:HRS_DM3AT-SF-PEJM5, symbol extra:DM3AT-SF-PEJM5
- added J?: Conn_01x02, symbol Connector_Generic:Conn_01x02
- added R10, R11, R12, R13, R7, R9: 4.7K, Resistor_SMD:R_0805_2012Metric, symbol Device:R
- added R8: 200k, Resistor_SMD:R_0805_2012Metric, symbol Device:R
- added SW1: SW_Push, Buttons_Switches_SMD:Panasonic_EVQPUJ_EVQPUA, symbol Switch:SW_Push
- added U2: TLV70218_SOT23-5, Package_TO_SOT_SMD:SOT-23-5, symbol Regulator_Linear:TLV70218_SOT23-5
- added U3: AP2112K-3.3, Package_TO_SOT_SMD:SOT-23-5, symbol Regulator_Linear:AP2112K-3.3
- added U4: MDBT50Q-1M, extra:MDBT50Q-1M, symbol extra:MDBT50Q-1M
- added U5: PCA9306, symbol Interface:PCA9306
- added U6: ICM-20948, extra:ICM-20948, symbol extra:ICM-20948
- added U7: BMP280, Package_LGA:Bosch_LGA-8_2x2.5mm_P0.65mm_ClockwisePinNumbering, symbol Sensor_Pressure:BMP280
- C1, C2: footprint (none) -> Capacitor_SMD:C_0805_2012Metric
- C4, C5, C7, C8: footprint (none) -> Capacitor_SMD:C_0603_1608Metric
- D1: footprint (none) -> Diodes_SMD:D_0805
- R1, R2: footprint (none) -> Resistor_SMD:R_0805_2012Metric
- R3, R4: footprint (none) -> Resistor_SMD:R_0603_1608Metric
- R5, R6: renamed from R?; footprint (none) -> Resistor_SMD:R_0805_2012Metric
- gave numbers to parts that had none: 2
Connections:
- net labels added: +1V8, +3V3, BMP_SCL, BMP_SDA, BUZZER, SCL_MPU, SDA_MPU, SD_CS, SD_MISO, SD_MOSI, SD_SCK, SWCLK, SWDIO, SWO
- net labels removed: TCK, TDI, TDO, TMS
- wire segments 32 -> 81
Other:
- moved on the sheet: C1, C2, C4, C5, C7, C8, D2, R3, R4, R5, R6, U1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

Commit message: started building board
Parts:
- removed Q1: Q_PMOS_DGS, symbol Device:Q_PMOS_DGS
- added Q1: Q_PMOS_GSD, digikey-footprints:SOT-23-3, symbol Device:Q_PMOS_GSD
- BZ1: footprint (none) -> Buzzer_Beeper:Buzzer_Murata_PKMCS0909E4000-R1
- C1, C3, C6: symbol Device:C -> Device:C_Small
- D2: footprint (none) -> Capacitor_SMD:C_0603_1608Metric
- J1: symbol Connector_Specialized:USB_B_Mini -> bed-sensor-rescue:USB_B_Mini-Connector_Specialized
- J2: symbol Connector_Specialized:Conn_ARM_JTAG_SWD_10 -> bed-sensor-rescue:Conn_ARM_JTAG_SWD_10-Connector_Specialized
- J4: renamed from J?; footprint (none) -> Connector_PinHeader_2.54mm:PinHeader_1x02_P2.54mm_Vertical
- R1, R10, R11, R12, R13, R2, R5, R6, R7, R8, R9: footprint Resistor_SMD:R_0805_2012Metric -> Fuse:Fuse_0603_1608Metric
- R3, R4: footprint Resistor_SMD:R_0603_1608Metric -> Fuse:Fuse_0603_1608Metric
- U5: footprint (none) -> Package_SO:VSSOP-8_2.3x2mm_P0.5mm
- Y1: footprint (none) -> OPL_Crystal_Oscillator:X2-SMD-3.2X1.5X0.55MM
Connections:
- wire segments 81 -> 83
Other:
- moved on the sheet: C3, C6

Commit message: updated schematic
Connections:
- net +1V8: no longer R12.2, R13.2
- net +3V3: now also R12.2, R13.2
Other:
- moved on the sheet: J4
Changed lines of the file:
@@
 	-1   0    0    1
-$EndComp
-$Comp
-L power:+1V8 #PWR0158
-U 1 1 5CA199C2
-P 9400 2900
-F 0 "#PWR0158" H 9400 2750 50  0001 C CNN
-F 1 "+1V8" H 9415 3073 50  0000 C CNN
-F 2 "" H 9400 2900 50  0001 C CNN
-F 3 "" H 9400 2900 50  0001 C CNN
-	1    9400 2900
-	1    0    0    -1
 $EndComp
 Wire Wire Line
@@
 L Connector_Generic:Conn_01x02 J4
 U 1 1 5CA96A5F
-P 2700 2400
-F 0 "J4" V 2664 2212 50  0000 R CNN
-F 1 "Conn_01x02" V 2573 2212 50  0000 R CNN
-F 2 "Connector_PinHeader_2.54mm:PinHeader_1x02_P2.54mm_Vertical" H 2700 2400 50  0001 C CNN
-F 3 "~" H 2700 2400 50  0001 C CNN
-	1    2700 2400
+P 2600 2450
+F 0 "J4" V 2564 2262 50  0000 R CNN
+F 1 "Conn_01x02" V 2750 2550 50  0000 R CNN
+F 2 "Connector_PinHeader_2.54mm:PinHeader_1x02_P2.54mm_Vertical" H 2600 2450 50  0001 C CNN
+F 3 "~" H 2600 2450 50  0001 C CNN
+	1    2600 2450
 	0    -1   -1   0
 $EndComp
@@
 L power:+BATT #PWR0165
 U 1 1 5CA98AFB
-P 2800 2600
-F 0 "#PWR0165" H 2800 2450 50  0001 C CNN
-F 1 "+BATT" H 2815 2773 50  0000 C CNN
-F 2 "" H 2800 2600 50  0001 C CNN
-F 3 "" H 2800 2600 50  0001 C CNN
-	1    2800 2600
+P 2700 2650
+F 0 "#PWR0165" H 2700 2500 50  0001 C CNN
+F 1 "+BATT" H 2550 2750 50  0000 C CNN
+F 2 "" H 2700 2650 50  0001 C CNN
+F 3 "" H 2700 2650 50  0001 C CNN
+	1    2700 2650
 	-1   0    0    1
 $EndComp
@@
 L power:GND #PWR0166
 U 1 1 5CA99901
-P 2700 2600
-F 0 "#PWR0166" H 2700 2350 50  0001 C CNN
-F 1 "GND" H 2705 2427 50  0000 C CNN
-F 2 "" H 2700 2600 50  0001 C CNN
-F 3 "" H 2700 2600 50  0001 C CNN
-	1    2700 2600
+P 2600 2650
+F 0 "#PWR0166" H 2600 2400 50  0001 C CNN
+F 1 "GND" H 2450 2550 50  0000 C CNN
+F 2 "" H 2600 2650 50  0001 C CNN
+F 3 "" H 2600 2650 50  0001 C CNN
+	1    2600 2650
 	1    0    0    -1
 $EndComp
@@
 Wire Wire Line
 	4400 4550 4500 4550
+$Comp
+L power:+3V3 #PWR?
+U 1 1 5CA00249
+P 9400 2900
+F 0 "#PWR?" H 9400 2750 50  0001 C CNN
+F 1 "+3V3" H 9415 3073 50  0000 C CNN
+F 2 "" H 9400 2900 50  0001 C CNN
+F 3 "" H 9400 2900 50  0001 C CNN
+	1    9400 2900
+	1    0    0    -1
+$EndComp
 $EndSCHEMATC

Commit message: moved pin
Connections:
- net SD_CS: now also U4.56 (P1.04); no longer U4.59 (P1.05)
Changed lines of the file:
@@
 Text GLabel 3550 3000 0    50   Input ~ 0
 SD_MISO
-Text GLabel 3550 2900 0    50   Input ~ 0
+Text GLabel 3550 2800 0    50   Input ~ 0
 SD_CS
 Text GLabel 3550 3100 0    50   Input ~ 0
@@
 	4400 4550 4500 4550
 $Comp
-L power:+3V3 #PWR?
+L power:+3V3 #PWR0158
 U 1 1 5CA00249
 P 9400 2900
-F 0 "#PWR?" H 9400 2750 50  0001 C CNN
+F 0 "#PWR0158" H 9400 2750 50  0001 C CNN
 F 1 "+3V3" H 9415 3073 50  0000 C CNN
 F 2 "" H 9400 2900 50  0001 C CNN

Commit message: updated kicad and vagrant file
Parts:
- J1: symbol bed-sensor-rescue:USB_B_Mini-Connector_Specialized -> bed-sensor-rescue:USB_B_Mini-Connector_Specialized-bed-sensor-rescue
- J2: symbol bed-sensor-rescue:Conn_ARM_JTAG_SWD_10-Connector_Specialized -> bed-sensor-rescue:Conn_ARM_JTAG_SWD_10-Connector_Specialized-bed-sensor-rescue
Changed lines of the file:
@@
 EESchema Schematic File Version 4
 LIBS:bed-sensor-cache
-EELAYER 26 0
+EELAYER 29 0
 EELAYER END
 $Descr A4 11693 8268
@@
 SDA_MPU
 $Comp
-L bed-sensor-rescue:USB_B_Mini-Connector_Specialized J1
+L bed-sensor-rescue:USB_B_Mini-Connector_Specialized-bed-sensor-rescue J1
 U 1 1 5CA6C0FF
 P 1100 5800
@@
 Connection ~ 1000 6200
 $Comp
-L bed-sensor-rescue:Conn_ARM_JTAG_SWD_10-Connector_Specialized J2
+L bed-sensor-rescue:Conn_ARM_JTAG_SWD_10-Connector_Specialized-bed-sensor-rescue J2
 U 1 1 5C9E80F8
 P 2950 6150

Commit message: updated footprints
Parts:
- R1, R10, R11, R12, R13, R2, R3, R4, R5, R6, R7, R8, R9: footprint Fuse:Fuse_0603_1608Metric -> Resistor_SMD:R_0603_1608Metric
- Y1: footprint OPL_Crystal_Oscillator:X2-SMD-3.2X1.5X0.55MM -> extra:FC-135 32.7680KA-AC3
Changed lines of the file:
@@
 F 0 "R2" H 1580 1654 50  0000 R CNN
 F 1 "100k" H 1580 1745 50  0000 R CNN
-F 2 "Fuse:Fuse_0603_1608Metric" V 1580 1700 50  0001 C CNN
+F 2 "Resistor_SMD:R_0603_1608Metric" V 1580 1700 50  0001 C CNN
 F 3 "~" H 1650 1700 50  0001 C CNN
 	1    1650 1700
@@
 F 0 "R1" H 920 1746 50  0000 L CNN
 F 1 "100K" H 920 1655 50  0000 L CNN
-F 2 "Fuse:Fuse_0603_1608Metric" V 780 1700 50  0001 C CNN
+F 2 "Resistor_SMD:R_0603_1608Metric" V 780 1700 50  0001 C CNN
 F 3 "~" H 850 1700 50  0001 C CNN
 	1    850  1700
@@
 F 0 "R3" V 5500 3550 50  0000 C CNN
 F 1 "22" V 5450 3400 50  0000 C CNN
-F 2 "Fuse:Fuse_0603_1608Metric" V 5380 3400 50  0001 C CNN
+F 2 "Resistor_SMD:R_0603_1608Metric" V 5380 3400 50  0001 C CNN
 F 3 "~" H 5450 3400 50  0001 C CNN
 	1    5450 3400
@@
 F 0 "R4" V 5500 3650 50  0000 C CNN
 F 1 "22" V 5450 3500 50  0000 C CNN
-F 2 "Fuse:Fuse_0603_1608Metric" V 5380 3500 50  0001 C CNN
+F 2 "Resistor_SMD:R_0603_1608Metric" V 5380 3500 50  0001 C CNN
 F 3 "~" H 5450 3500 50  0001 C CNN
 	1    5450 3500
@@
 F 0 "Y1" V 5654 2431 50  0000 L CNN
 F 1 "32.768" V 5950 2150 50  0000 L CNN
-F 2 "OPL_Crystal_Oscillator:X2-SMD-3.2X1.5X0.55MM" H 5700 2300 50  0001 C CNN
+F 2 "extra:FC-135 32.7680KA-AC3" H 5700 2300 50  0001 C CNN
 F 3 "~" H 5700 2300 50  0001 C CNN
 	1    5700 2300
@@
 F 0 "R6" H 2170 2796 50  0000 L CNN
 F 1 "1K" H 2170 2705 50  0000 L CNN
-F 2 "Fuse:Fuse_0603_1608Metric" V 2030 2750 50  0001 C CNN
+F 2 "Resistor_SMD:R_0603_1608Metric" V 2030 2750 50  0001 C CNN
 F 3 "~" H 2100 2750 50  0001 C CNN
 	1    2100 2750
@@
 F 0 "R5" V 943 2600 50  0000 C CNN
 F 1 "4.7k" V 1034 2600 50  0000 C CNN
-F 2 "Fuse:Fuse_0603_1608Metric" V 1080 2600 50  0001 C CNN
+F 2 "Resistor_SMD:R_0603_1608Metric" V 1080 2600 50  0001 C CNN
 F 3 "~" H 1150 2600 50  0001 C CNN
 	1    1150 2600
@@
 F 0 "R9" H 7520 1546 50  0000 L CNN
 F 1 "4.7K" H 7520 1455 50  0000 L CNN
-F 2 "Fuse:Fuse_0603_1608Metric" V 7380 1500 50  0001 C CNN
+F 2 "Resistor_SMD:R_0603_1608Metric" V 7380 1500 50  0001 C CNN
 F 3 "~" H 7450 1500 50  0001 C CNN
 	1    7450 1500
@@
 F 0 "R7" H 7170 1546 50  0000 L CNN
 F 1 "4.7K" H 7170 1455 50  0000 L CNN
-F 2 "Fuse:Fuse_0603_1608Metric" V 7030 1500 50  0001 C CNN
+F 2 "Resistor_SMD:R_0603_1608Metric" V 7030 1500 50  0001 C CNN
 F 3 "~" H 7100 1500 50  0001 C CNN
 	1    7100 1500
@@
 F 0 "R11" H 8820 1496 50  0000 L CNN
 F 1 "4.7K" H 8820 1405 50  0000 L CNN
-F 2 "Fuse:Fuse_0603_1608Metric" V 8680 1450 50  0001 C CNN
+F 2 "Resistor_SMD:R_0603_1608Metric" V 8680 1450 50  0001 C CNN
 F 3 "~" H 8750 1450 50  0001 C CNN
 	1    8750 1450
@@
 F 0 "R10" H 8470 1496 50  0000 L CNN
 F 1 "4.7K" H 8470 1405 50  0000 L CNN
-F 2 "Fuse:Fuse_0603_1608Metric" V 8330 1450 50  0001 C CNN
+F 2 "Resistor_SMD:R_0603_1608Metric" V 8330 1450 50  0001 C CNN
 F 3 "~" H 8400 1450 50  0001 C CNN
 	1    8400 1450
@@
 F 0 "R8" H 7320 2846 50  0000 L CNN
 F 1 "200k" H 7320 2755 50  0000 L CNN
-F 2 "Fuse:Fuse_0603_1608Metric" V 7180 2800 50  0001 C CNN
+F 2 "Resistor_SMD:R_0603_1608Metric" V 7180 2800 50  0001 C CNN
 F 3 "~" H 7250 2800 50  0001 C CNN
 	1    7250 2800
@@
 F 0 "R13" H 9470 3246 50  0000 L CNN
 F 1 "4.7K" H 9470 3155 50  0000 L CNN
-F 2 "Fuse:Fuse_0603_1608Metric" V 9330 3200 50  0001 C CNN
+F 2 "Resistor_SMD:R_0603_1608Metric" V 9330 3200 50  0001 C CNN
 F 3 "~" H 9400 3200 50  0001 C CNN
 	1    9400 3200
@@
 F 0 "R12" H 9120 3246 50  0000 L CNN
 F 1 "4.7K" H 9120 3155 50  0000 L CNN
-F 2 "Fuse:Fuse_0603_1608Metric" V 8980 3200 50  0001 C CNN
+F 2 "Resistor_SMD:R_0603_1608Metric" V 8980 3200 50  0001 C CNN
 F 3 "~" H 9050 3200 50  0001 C CNN
 	1    9050 3200

Commit message: finalized order list
Parts:
- added D3: LED_RCGB, LED_SMD:LED_Kingbright_AAA3528ESGCT, symbol Device:LED_RCGB
- added R14, R15, R16: 330, Resistor_SMD:R_0603_1608Metric, symbol Device:R
- added R17, R18: 100k, Resistor_SMD:R_0603_1608Metric, symbol Device:R
- D1: footprint Diodes_SMD:D_0805 -> Diode_SMD:D_SOD-123
- D2: footprint Capacitor_SMD:C_0603_1608Metric -> Diode_SMD:D_0603_1608Metric
- J1: footprint Connectors:USB_Mini-B -> digikey-footprints:USB_Micro_B_Female_10118194-0001LF; symbol bed-sensor-rescue:USB_B_Mini-Connector_Specialized-bed-sensor-rescue -> bed-sensor-rescue:USB_B_Mini-Connector_Specialized-bed-sensor-rescue-bed-sensor-rescue
- J2: symbol bed-sensor-rescue:Conn_ARM_JTAG_SWD_10-Connector_Specialized-bed-sensor-rescue -> bed-sensor-rescue:Conn_ARM_JTAG_SWD_10-Connector_Specialized-bed-sensor-rescue-bed-sensor-rescue
Connections:
- net +BATT: now also R17.1
- net BMP_SDA: now also U4.44 (P0.20); no longer U4.36 (P0.14)
- net GND: now also D3.2 (K), R18.2
- net SD_MISO: now also U4.38 (P0.16); no longer U4.57 (P1.06)
- net SD_MOSI: now also U4.43 (P0.21); no longer U4.58 (P1.07)
- net VDIV: now reaches U4.20 (P0.04/AIN2)
- net VDIV: now also R17.2, R18.1
- net B_LED: now reaches U4.4 (P1.11)
- net B_LED: now also R16.1
- net R_LED: now reaches U4.6 (P1.13)
- net R_LED: now also R14.1
- net G_LED: now reaches U4.8 (P1.15)
- net G_LED: now also R15.1
- new net: D3.1 (RA), R14.2
- new net: D3.3 (GA), R15.2
- new net: D3.4 (BA), R16.2
Changed lines of the file:
@@
 EESchema Schematic File Version 4
 LIBS:bed-sensor-cache
-EELAYER 29 0
+EELAYER 26 0
 EELAYER END
 $Descr A4 11693 8268
@@
 F 0 "D1" H 1250 1234 50  0000 C CNN
 F 1 "D_Schottky" H 1250 1325 50  0000 C CNN
-F 2 "Diodes_SMD:D_0805" H 1250 1450 50  0001 C CNN
+F 2 "Diode_SMD:D_SOD-123" H 1250 1450 50  0001 C CNN
 F 3 "~" H 1250 1450 50  0001 C CNN
 	1    1250 1450
@@
 F 0 "D2" V 2045 3128 50  0000 L CNN
 F 1 "LED" V 2136 3128 50  0000 L CNN
-F 2 "Capacitor_SMD:C_0603_1608Metric" H 2100 3050 50  0001 C CNN
+F 2 "Diode_SMD:D_0603_1608Metric" H 2100 3050 50  0001 C CNN
 F 3 "~" H 2100 3050 50  0001 C CNN
 	1    2100 3050
@@
 SDA_MPU
 $Comp
-L bed-sensor-rescue:USB_B_Mini-Connector_Specialized-bed-sensor-rescue J1
+L bed-sensor-rescue:USB_B_Mini-Connector_Specialized-bed-sensor-rescue-bed-sensor-rescue J1
 U 1 1 5CA6C0FF
 P 1100 5800
 F 0 "J1" H 1157 6267 50  0000 C CNN
 F 1 "USB_B_Mini" H 1157 6176 50  0000 C CNN
-F 2 "Connectors:USB_Mini-B" H 1250 5750 50  0001 C CNN
+F 2 "digikey-footprints:USB_Micro_B_Female_10118194-0001LF" H 1250 5750 50  0001 C CNN
 F 3 "~" H 1250 5750 50  0001 C CNN
 	1    1100 5800
@@
 Connection ~ 1000 6200
 $Comp
-L bed-sensor-rescue:Conn_ARM_JTAG_SWD_10-Connector_Specialized-bed-sensor-rescue J2
+L bed-sensor-rescue:Conn_ARM_JTAG_SWD_10-Connector_Specialized-bed-sensor-rescue-bed-sensor-rescue J2
 U 1 1 5C9E80F8
 P 2950 6150
@@
 	0    -1   -1   0
 $EndComp
-Text GLabel 3550 3000 0    50   Input ~ 0
+Text GLabel 3550 1800 0    50   Input ~ 0
 SD_MISO
 Text GLabel 3550 2800 0    50   Input ~ 0
 SD_CS
-Text GLabel 3550 3100 0    50   Input ~ 0
+Text GLabel 3550 2100 0    50   Input ~ 0
 SD_MOSI
 Text GLabel 3550 3200 0    50   Input ~ 0
@@
 Text GLabel 3550 1500 0    50   Input ~ 0
 BMP_SCL
-Text GLabel 3550 1600 0    50   Input ~ 0
+Text GLabel 3550 2000 0    50   Input ~ 0
 BMP_SDA
 $Comp
@@
 	1    0    0    -1
 $EndComp
+$Comp
+L Device:LED_RCGB D3
+U 1 1 5CA5A38C
+P 5800 5600
+F 0 "D3" V 5846 5270 50  0000 R CNN
+F 1 "LED_RCGB" V 5755 5270 50  0000 R CNN
+F 2 "LED_SMD:LED_Kingbright_AAA3528ESGCT" H 5800 5550 50  0001 C CNN
+F 3 "~" H 5800 5550 50  0001 C CNN
+	1    5800 5600
+	0    -1   -1   0
+$EndComp
+$Comp
+L Device:R R14
+U 1 1 5CA6159F
+P 5600 5250
+F 0 "R14" H 5670 5296 50  0000 L CNN
+F 1 "330" H 5670 5205 50  0000 L CNN
+F 2 "Resistor_SMD:R_0603_1608Metric" V 5530 5250 50  0001 C CNN
+F 3 "~" H 5600 5250 50  0001 C CNN
+	1    5600 5250
+	1    0    0    -1
+$EndComp
+$Comp
+L Device:R R15
+U 1 1 5CA636F3
+P 5800 5250
+F 0 "R15" H 5870 5296 50  0000 L CNN
+F 1 "330" H 5870 5205 50  0000 L CNN
+F 2 "Resistor_SMD:R_0603_1608Metric" V 5730 5250 50  0001 C CNN
+F 3 "~" H 5800 5250 50  0001 C CNN
+	1    5800 5250
+	1    0    0    -1
+$EndComp
+$Comp
+L Device:R R16
+U 1 1 5CA63769
+P 6000 5250
+F 0 "R16" H 6070 5296 50  0000 L CNN
+F 1 "330" H 6070 5205 50  0000 L CNN
+F 2 "Resistor_SMD:R_0603_1608Metric" V 5930 5250 50  0001 C CNN
+F 3 "~" H 6000 5250 50  0001 C CNN
+	1    6000 5250
+	1    0    0    -1
+$EndComp
+Text GLabel 3550 3600 0    50   Input ~ 0
+R_LED
+Text GLabel 3550 3800 0    50   Input ~ 0
+G_LED
+Text GLabel 3550 3400 0    50   Input ~ 0
+B_LED
+$Comp
+L power:GND #PWR0167
+U 1 1 5CA63A2B
+P 5800 5800
+F 0 "#PWR0167" H 5800 5550 50  0001 C CNN
+F 1 "GND" H 5805 5627 50  0000 C CNN
+F 2 "" H 5800 5800 50  0001 C CNN
+F 3 "" H 5800 5800 50  0001 C CNN
+	1    5800 5800
+	1    0    0    -1
+$EndComp
+Text GLabel 5600 5100 1    50   Input ~ 0
+R_LED
+Text GLabel 5800 5100 1    50   Input ~ 0
+G_LED
+Text GLabel 6000 5100 1    50   Input ~ 0
+B_LED
+$Comp
+L Device:R R17
+U 1 1 5CA79672
+P 7150 5050
+F 0 "R17" H 7220 5096 50  0000 L CNN
+F 1 "100k" H 7220 5005 50  0000 L CNN
+F 2 "Resistor_SMD:R_0603_1608Metric" V 7080 5050 50  0001 C CNN
+F 3 "~" H 7150 5050 50  0001 C CNN
+	1    7150 5050
+	1    0    0    -1
+$EndComp
+$Comp
+L Device:R R18
+U 1 1 5CA796FA
+P 7150 5350
+F 0 "R18" H 7220 5396 50  0000 L CNN
+F 1 "100k" H 7220 5305 50  0000 L CNN
+F 2 "Resistor_SMD:R_0603_1608Metric" V 7080 5350 50  0001 C CNN
+F 3 "~" H 7150 5350 50  0001 C CNN
+	1    7150 5350
+	1    0    0    -1
+$EndComp
+$Comp
+L power:+BATT #PWR0168
+U 1 1 5CA7B569
+P 7150 4900
+F 0 "#PWR0168" H 7150 4750 50  0001 C CNN
+F 1 "+BATT" H 7165 5073 50  0000 C CNN
+F 2 "" H 7150 4900 50  0001 C CNN
+F 3 "" H 7150 4900 50  0001 C CNN
+	1    7150 4900
+	1    0    0    -1
+$EndComp
+$Comp
+L power:GND #PWR0169
+U 1 1 5CA7B666
+P 7150 5500
+F 0 "#PWR0169" H 7150 5250 50  0001 C CNN
+F 1 "GND" H 7155 5327 50  0000 C CNN
+F 2 "" H 7150 5500 50  0001 C CNN
+F 3 "" H 7150 5500 50  0001 C CNN
+	1    7150 5500
+	1    0    0    -1
+$EndComp
+Text GLabel 7550 5200 2    50   Input ~ 0
+VDIV
+Wire Wire Line
+	7150 5200 7550 5200
+Connection ~ 7150 5200
+Text GLabel 5300 3050 2    50   Input ~ 0
+VDIV
 $EndSCHEMATC

Commit message: update layout
Parts:
- removed D3: LED_RCGB, LED_SMD:LED_Kingbright_AAA3528ESGCT, symbol Device:LED_RCGB
- removed R14, R15, R16: 330, Resistor_SMD:R_0603_1608Metric, symbol Device:R
- added D3: WS2812B, LED_SMD:LED_WS2812B_PLCC4_5.0x5.0mm_P3.2mm, symbol LED:WS2812B
- J1: symbol bed-sensor-rescue:USB_B_Mini-Connector_Specialized-bed-sensor-rescue-bed-sensor-rescue -> bed-sensor-rescue:USB_B_Mini-Connector_Specialized-bed-sensor-rescue-bed-sensor-rescue-bed-sensor-rescue
- J2: symbol bed-sensor-rescue:Conn_ARM_JTAG_SWD_10-Connector_Specialized-bed-sensor-rescue-bed-sensor-rescue -> bed-sensor-rescue:Conn_ARM_JTAG_SWD_10-Connector_Specialized-bed-sensor-rescue-bed-sensor-rescue-bed-sensor-rescue
- R17, R18: value 100k -> 100K
Connections:
- net +3V3: now also D3.1 (VDD)
- net GND: now also D3.3 (VSS)
- net B_LED: no longer names the net of U4.4 (P1.11)
- net G_LED renamed NEO_LED
- net NEO_LED: now also D3.4 (DIN)
- net R_LED: no longer names the net of U4.6 (P1.13)
Changed lines of the file:
@@
 EESchema Schematic File Version 4
 LIBS:bed-sensor-cache
-EELAYER 26 0
+EELAYER 29 0
 EELAYER END
 $Descr A4 11693 8268
@@
 SDA_MPU
 $Comp
-L bed-sensor-rescue:USB_B_Mini-Connector_Specialized-bed-sensor-rescue-bed-sensor-rescue J1
+L bed-sensor-rescue:USB_B_Mini-Connector_Specialized-bed-sensor-rescue-bed-sensor-rescue-bed-sensor-rescue J1
 U 1 1 5CA6C0FF
 P 1100 5800
@@
 Connection ~ 1000 6200
 $Comp
-L bed-sensor-rescue:Conn_ARM_JTAG_SWD_10-Connector_Specialized-bed-sensor-rescue-bed-sensor-rescue J2
+L bed-sensor-rescue:Conn_ARM_JTAG_SWD_10-Connector_Specialized-bed-sensor-rescue-bed-sensor-rescue-bed-sensor-rescue J2
 U 1 1 5C9E80F8
 P 2950 6150
@@
 	1    0    0    -1
 $EndComp
-$Comp
-L Device:LED_RCGB D3
-U 1 1 5CA5A38C
-P 5800 5600
-F 0 "D3" V 5846 5270 50  0000 R CNN
-F 1 "LED_RCGB" V 5755 5270 50  0000 R CNN
-F 2 "LED_SMD:LED_Kingbright_AAA3528ESGCT" H 5800 5550 50  0001 C CNN
-F 3 "~" H 5800 5550 50  0001 C CNN
-	1    5800 5600
-	0    -1   -1   0
-$EndComp
-$Comp
-L Device:R R14
-U 1 1 5CA6159F
-P 5600 5250
-F 0 "R14" H 5670 5296 50  0000 L CNN
-F 1 "330" H 5670 5205 50  0000 L CNN
-F 2 "Resistor_SMD:R_0603_1608Metric" V 5530 5250 50  0001 C CNN
-F 3 "~" H 5600 5250 50  0001 C CNN
-	1    5600 5250
-	1    0    0    -1
-$EndComp
-$Comp
-L Device:R R15
-U 1 1 5CA636F3
-P 5800 5250
-F 0 "R15" H 5870 5296 50  0000 L CNN
-F 1 "330" H 5870 5205 50  0000 L CNN
-F 2 "Resistor_SMD:R_0603_1608Metric" V 5730 5250 50  0001 C CNN
-F 3 "~" H 5800 5250 50  0001 C CNN
-	1    5800 5250
-	1    0    0    -1
-$EndComp
-$Comp
-L Device:R R16
-U 1 1 5CA63769
-P 6000 5250
-F 0 "R16" H 6070 5296 50  0000 L CNN
-F 1 "330" H 6070 5205 50  0000 L CNN
-F 2 "Resistor_SMD:R_0603_1608Metric" V 5930 5250 50  0001 C CNN
-F 3 "~" H 6000 5250 50  0001 C CNN
-	1    6000 5250
-	1    0    0    -1
-$EndComp
-Text GLabel 3550 3600 0    50   Input ~ 0
-R_LED
-Text GLabel 3550 3800 0    50   Input ~ 0
-G_LED
-Text GLabel 3550 3400 0    50   Input ~ 0
-B_LED
-$Comp
-L power:GND #PWR0167
-U 1 1 5CA63A2B
-P 5800 5800
-F 0 "#PWR0167" H 5800 5550 50  0001 C CNN
-F 1 "GND" H 5805 5627 50  0000 C CNN
-F 2 "" H 5800 5800 50  0001 C CNN
-F 3 "" H 5800 5800 50  0001 C CNN
-	1    5800 5800
-	1    0    0    -1
-$EndComp
-Text GLabel 5600 5100 1    50   Input ~ 0
-R_LED
-Text GLabel 5800 5100 1    50   Input ~ 0
-G_LED
-Text GLabel 6000 5100 1    50   Input ~ 0
-B_LED
+Text GLabel 5500 5500 0    50   Input ~ 0
+NEO_LED
 $Comp
 L Device:R R17
@@
 P 7150 5050
 F 0 "R17" H 7220 5096 50  0000 L CNN
-F 1 "100k" H 7220 5005 50  0000 L CNN
+F 1 "100K" H 7220 5005 50  0000 L CNN
 F 2 "Resistor_SMD:R_0603_1608Metric" V 7080 5050 50  0001 C CNN
 F 3 "~" H 7150 5050 50  0001 C CNN
@@
 P 7150 5350
 F 0 "R18" H 7220 5396 50  0000 L CNN
-F 1 "100k" H 7220 5305 50  0000 L CNN
+F 1 "100K" H 7220 5305 50  0000 L CNN
 F 2 "Resistor_SMD:R_0603_1608Metric" V 7080 5350 50  0001 C CNN
 F 3 "~" H 7150 5350 50  0001 C CNN
@@
 Text GLabel 5300 3050 2    50   Input ~ 0
 VDIV
+$Comp
+L LED:WS2812B D3
+U 1 1 5CB862BC
+P 5800 5500
+F 0 "D3" H 6144 5546 50  0000 L CNN
+F 1 "WS2812B" H 6144 5455 50  0000 L CNN
+F 2 "LED_SMD:LED_WS2812B_PLCC4_5.0x5.0mm_P3.2mm" H 5850 5200 50  0001 L TNN
+F 3 "https://cdn-shop.adafruit.com/datasheets/WS2812B.pdf" H 5900 5125 50  0001 L TNN
+	1    5800 5500
+	1    0    0    -1
+$EndComp
+$Comp
+L power:+3.3V #PWR0167
+U 1 1 5CB891BF
+P 5800 5200
+F 0 "#PWR0167" H 5800 5050 50  0001 C CNN
+F 1 "+3.3V" H 5815 5373 50  0000 C CNN
+F 2 "" H 5800 5200 50  0001 C CNN
+F 3 "" H 5800 5200 50  0001 C CNN
+	1    5800 5200
+	1    0    0    -1
+$EndComp
+$Comp
+L power:GND #PWR0170
+U 1 1 5CB89DBA
+P 5800 5800
+F 0 "#PWR0170" H 5800 5550 50  0001 C CNN
+F 1 "GND" H 5805 5627 50  0000 C CNN
+F 2 "" H 5800 5800 50  0001 C CNN
+F 3 "" H 5800 5800 50  0001 C CNN
+	1    5800 5800
+	1    0    0    -1
+$EndComp
+Text GLabel 3550 3800 0    50   Input ~ 0
+NEO_LED
 $EndSCHEMATC
