File: hardware/bed-sensor.sch (KiCad schematic (older format))
At the start: 49 parts, among them J1 USB_B_Mini, J2 Conn_ARM_JTAG_SWD_10, J3 DM3AT-SF-PEJM5, J4 Conn_01x02, Q1 Q_PMOS_GSD, SW1 SW_Push, U1 MCP73831-2-OT, U2 TLV70218_SOT23-5, U3 AP2112K-3.3, U4 MDBT50Q-1M, U5 PCA9306, U6 ICM-20948, U7 BMP280, Y1 32.768

Commit message: added bom file
Parts:
- R2: value 100k -> 100K
- R5: value 4.7k -> 4.7K
Changed lines of the file:
@@
 AR Path="/5C947A0A/5C948E09" Ref="R?"  Part="1"
 F 0 "R2" H 1580 1654 50  0000 R CNN
-F 1 "100k" H 1580 1745 50  0000 R CNN
+F 1 "100K" H 1580 1745 50  0000 R CNN
 F 2 "Resistor_SMD:R_0603_1608Metric" V 1580 1700 50  0001 C CNN
 F 3 "~" H 1650 1700 50  0001 C CNN
@@
 P 1150 2600
 F 0 "R5" V 943 2600 50  0000 C CNN
-F 1 "4.7k" V 1034 2600 50  0000 C CNN
+F 1 "4.7K" V 1034 2600 50  0000 C CNN
 F 2 "Resistor_SMD:R_0603_1608Metric" V 1080 2600 50  0001 C CNN
 F 3 "~" H 1150 2600 50  0001 C CNN

Commit message: updated schematic
Parts:
- J1: symbol bed-sensor-rescue:USB_B_Mini-Connector_Specialized-bed-sensor-rescue-bed-sensor-rescue-bed-sensor-rescue -> bed-sensor-rescue:USB_B_Mini-Connector_Specialized-bed-sensor-rescue-bed-sensor-rescue-bed-sensor-rescue-bed-sensor-res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
- J2: symbol bed-sensor-rescue:Conn_ARM_JTAG_SWD_10-Connector_Specialized-bed-sensor-rescue-bed-sensor-rescue-bed-sensor-rescue -> bed-sensor-rescue:Conn_ARM_JTAG_SWD_10-Connector_Specialized-bed-sensor-rescue-bed-sensor-rescue-bed-sensor-rescue-bed-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
Changed lines of the file:
@@
 EESchema Schematic File Version 4
 LIBS:bed-sensor-cache
-EELAYER 29 0
+EELAYER 26 0
 EELAYER END
 $Descr A4 11693 8268
@@
 SDA_MPU
 $Comp
-L bed-sensor-rescue:USB_B_Mini-Connector_Specialized-bed-sensor-rescue-bed-sensor-rescue-bed-sensor-rescue J1
+L bed-sensor-rescue:USB_B_Mini-Connector_Specialized-bed-sensor-rescue-bed-sensor-rescue-bed-sensor-rescue-bed-sensor-rescue J1
 U 1 1 5CA6C0FF
 P 1100 5800
@@
 Connection ~ 1000 6200
 $Comp
-L bed-sensor-rescue:Conn_ARM_JTAG_SWD_10-Connector_Specialized-bed-sensor-rescue-bed-sensor-rescue-bed-sensor-rescue J2
+L bed-sensor-rescue:Conn_ARM_JTAG_SWD_10-Connector_Specialized-bed-sensor-rescue-bed-sensor-rescue-bed-sensor-rescue-bed-sensor-rescue J2
 U 1 1 5C9E80F8
 P 2950 6150

Commit message: removed extra
Parts:
- J1: symbol bed-sensor-rescue:USB_B_Mini-Connector_Specialized-bed-sensor-rescue-bed-sensor-rescue-bed-sensor-rescue-bed-sensor-rescue -> bed-sensor-rescue:USB_B_Mini-Connector_Specialized-bed-sensor-rescue-bed-sensor-rescue-bed-sensor-rescue-bed-sensor-rescue-bed-sensor-rescue
- J2: symbol bed-sensor-rescue:Conn_ARM_JTAG_SWD_10-Connector_Specialized-bed-sensor-rescue-bed-sensor-rescue-bed-sensor-rescue-bed-sensor-rescue -> bed-sensor-rescue:Conn_ARM_JTAG_SWD_10-Connector_Specialized-bed-sensor-rescue-bed-sensor-rescue-bed-sensor-rescue-bed-sensor-rescue-bed-sensor-rescue
Changed lines of the file:
@@
 EESchema Schematic File Version 4
 LIBS:bed-sensor-cache
-EELAYER 26 0
+EELAYER 29 0
 EELAYER END
 $Descr A4 11693 8268
@@
 SDA_MPU
 $Comp
-L bed-sensor-rescue:USB_B_Mini-Connector_Specialized-bed-sensor-rescue-bed-sensor-rescue-bed-sensor-rescue-bed-sensor-rescue J1
+L bed-sensor-rescue:USB_B_Mini-Connector_Specialized-bed-sensor-rescue-bed-sensor-rescue-bed-sensor-rescue-bed-sensor-rescue-bed-sensor-rescue J1
 U 1 1 5CA6C0FF
 P 1100 5800
@@
 Connection ~ 1000 6200
 $Comp
-L bed-sensor-rescue:Conn_ARM_JTAG_SWD_10-Connector_Specialized-bed-sensor-rescue-bed-sensor-rescue-bed-sensor-rescue-bed-sensor-rescue J2
+L bed-sensor-rescue:Conn_ARM_JTAG_SWD_10-Connector_Specialized-bed-sensor-rescue-bed-sensor-rescue-bed-sensor-rescue-bed-sensor-rescue-bed-sensor-rescue J2
 U 1 1 5C9E80F8
 P 2950 6150

Commit message: added drivers and board
Parts:
- J1: symbol bed-sensor-rescue:USB_B_Mini-Connector_Specialized-bed-sensor-rescue-bed-sensor-rescue-bed-sensor-rescue-bed-sensor-rescue-bed-sensor-rescue -> bed-sensor-rescue:USB_B_Mini-Connector_Specialized-bed-sensor-rescue-bed-sensor-rescue-bed-sensor-rescue-bed-sensor-rescue-bed-sensor-rescue-bed-sensor-rescue
- J2: symbol bed-sensor-rescue:Conn_ARM_JTAG_SWD_10-Connector_Specialized-bed-sensor-rescue-bed-sensor-rescue-bed-sensor-rescue-bed-sensor-rescue-bed-sensor-rescue -> bed-sensor-rescue:Conn_ARM_JTAG_SWD_10-Connector_Specialized-bed-sensor-rescue-bed-sensor-rescue-bed-sensor-rescue-bed-sensor-rescue-bed-sensor-rescue-bed-sensor-rescue
Changed lines of the file:
@@
 EESchema Schematic File Version 4
 LIBS:bed-sensor-cache
-EELAYER 29 0
+EELAYER 26 0
 EELAYER END
 $Descr A4 11693 8268
@@
 SDA_MPU
 $Comp
-L bed-sensor-rescue:USB_B_Mini-Connector_Specialized-bed-sensor-rescue-bed-sensor-rescue-bed-sensor-rescue-bed-sensor-rescue-bed-sensor-rescue J1
+L bed-sensor-rescue:USB_B_Mini-Connector_Specialized-bed-sensor-rescue-bed-sensor-rescue-bed-sensor-rescue-bed-sensor-rescue-bed-sensor-rescue-bed-sensor-rescue J1
 U 1 1 5CA6C0FF
 P 1100 5800
@@
 Connection ~ 1000 6200
 $Comp
-L bed-sensor-rescue:Conn_ARM_JTAG_SWD_10-Connector_Specialized-bed-sensor-rescue-bed-sensor-rescue-bed-sensor-rescue-bed-sensor-rescue-bed-sensor-rescue J2
+L bed-sensor-rescue:Conn_ARM_JTAG_SWD_10-Connector_Specialized-bed-sensor-rescue-bed-sensor-rescue-bed-sensor-rescue-bed-sensor-rescue-bed-sensor-rescue-bed-sensor-rescue J2
 U 1 1 5C9E80F8
 P 2950 6150

Commit message: updated board
Parts:
- J1: symbol bed-sensor-rescue:USB_B_Mini-Connector_Specialized-bed-sensor-rescue-bed-sensor-rescue-bed-sensor-rescue-bed-sensor-rescue-bed-sensor-rescue-bed-sensor-rescue -> bed-sensor-rescue:USB_B_Mini-Connector_Specialized-bed-sensor-rescue-bed-sensor-rescue-bed-sensor-rescue-bed-sensor-rescue-bed-sensor-rescue-bed-sensor-rescue-bed-sensor-rescue
- J2: symbol bed-sensor-rescue:Conn_ARM_JTAG_SWD_10-Connector_Specialized-bed-sensor-rescue-bed-sensor-rescue-bed-sensor-rescue-bed-sensor-rescue-bed-sensor-rescue-bed-sensor-rescue -> bed-sensor-rescue:Conn_ARM_JTAG_SWD_10-Connector_Specialized-bed-sensor-rescue-bed-sensor-rescue-bed-sensor-rescue-bed-sensor-rescue-bed-sensor-rescue-bed-sensor-rescue-bed-sensor-rescue
Changed lines of the file:
@@
 SDA_MPU
 $Comp
-L bed-sensor-rescue:USB_B_Mini-Connector_Specialized-bed-sensor-rescue-bed-sensor-rescue-bed-sensor-rescue-bed-sensor-rescue-bed-sensor-rescue-bed-sensor-rescue J1
+L bed-sensor-rescue:USB_B_Mini-Connector_Specialized-bed-sensor-rescue-bed-sensor-rescue-bed-sensor-rescue-bed-sensor-rescue-bed-sensor-rescue-bed-sensor-rescue-bed-sensor-rescue J1
 U 1 1 5CA6C0FF
 P 1100 5800
@@
 Connection ~ 1000 6200
 $Comp
-L bed-sensor-rescue:Conn_ARM_JTAG_SWD_10-Connector_Specialized-bed-sensor-rescue-bed-sensor-rescue-bed-sensor-rescue-bed-sensor-rescue-bed-sensor-rescue-bed-sensor-rescue J2
+L bed-sensor-rescue:Conn_ARM_JTAG_SWD_10-Connector_Specialized-bed-sensor-rescue-bed-sensor-rescue-bed-sensor-rescue-bed-sensor-rescue-bed-sensor-rescue-bed-sensor-rescue-bed-sensor-rescue J2
 U 1 1 5C9E80F8
 P 2950 6150

Commit message: updated dts for pressure sensor
Parts:
- J1: symbol bed-sensor-rescue:USB_B_Mini-Connector_Specialized-bed-sensor-rescue-bed-sensor-rescue-bed-sensor-rescue-bed-sensor-rescue-bed-sensor-rescue-bed-sensor-rescue-bed-sensor-rescue -> bed-sensor-rescue:USB_B_Mini-Connector_Specialized-bed-sensor-rescue-bed-sensor-rescue-bed-sensor-rescue-bed-sensor-rescue-bed-sensor-rescue-bed-sensor-rescue-bed-sensor-rescue-bed-sensor-rescue
- J2: symbol bed-sensor-rescue:Conn_ARM_JTAG_SWD_10-Connector_Specialized-bed-sensor-rescue-bed-sensor-rescue-bed-sensor-rescue-bed-sensor-rescue-bed-sensor-rescue-bed-sensor-rescue-bed-sensor-rescue -> bed-sensor-rescue:Conn_ARM_JTAG_SWD_10-Connector_Specialized-bed-sensor-rescue-bed-sensor-rescue-bed-sensor-rescue-bed-sensor-rescue-bed-sensor-rescue-bed-sensor-rescue-bed-sensor-rescue-bed-sensor-rescue
Changed lines of the file:
@@
 SDA_MPU
 $Comp
-L bed-sensor-rescue:USB_B_Mini-Connector_Specialized-bed-sensor-rescue-bed-sensor-rescue-bed-sensor-rescue-bed-sensor-rescue-bed-sensor-rescue-bed-sensor-rescue-bed-sensor-rescue J1
+L bed-sensor-rescue:USB_B_Mini-Connector_Specialized-bed-sensor-rescue-bed-sensor-rescue-bed-sensor-rescue-bed-sensor-rescue-bed-sensor-rescue-bed-sensor-rescue-bed-sensor-rescue-bed-sensor-rescue J1
 U 1 1 5CA6C0FF
 P 1100 5800
@@
 Connection ~ 1000 6200
 $Comp
-L bed-sensor-rescue:Conn_ARM_JTAG_SWD_10-Connector_Specialized-bed-sensor-rescue-bed-sensor-rescue-bed-sensor-rescue-bed-sensor-rescue-bed-sensor-rescue-bed-sensor-rescue-bed-sensor-rescue J2
+L bed-sensor-rescue:Conn_ARM_JTAG_SWD_10-Connector_Specialized-bed-sensor-rescue-bed-sensor-rescue-bed-sensor-rescue-bed-sensor-rescue-bed-sensor-rescue-bed-sensor-rescue-bed-sensor-rescue-bed-sensor-rescue J2
 U 1 1 5C9E80F8
 P 2950 6150
